File: KL27Z_breakout.sch (KiCad schematic (older format))
At the start: 15 parts, among them J1 USB_mini_micro_B, P1 CONN_01X08, P2 CONN_01X08, P3 CONN_01X08, P4 CONN_01X08, SW1 SW_PUSH, SW2 SW_PUSH, U1 MKL27Z256VFM4

Commit message: 400mil pcb
Parts:
- removed P1, P4: CONN_01X08, symbol CONN_01X08
- added P1, P4: CONN_01X06, symbol CONN_01X06
Connections:
- net GND: now also P3.8 (P8), P4.6 (P6)
- net PTC4: now also P4.1 (P1); no longer P3.8 (P8)
- net PTC5: now also P4.2 (P2)
- net PTC6: now also P4.3 (P3)
- net PTC7: now also P4.4 (P4)
- net PTD4: now also P4.5 (P5)
- net PTD5: now also P1.3 (P3)
- net PTD6: now also P1.4 (P4)
- net PTD7: now also P1.5 (P5)
- net PTE0: now also P1.6 (P6)
- net VBUS: now also P1.1 (P1)
- net VREGIN: now also P1.2 (P2)
Changed lines of the file:
@@
 Text Notes 1400 4175 0    60   ~ 0
 External power option
-Text Notes 4050 4100 2    60   ~ 12
+Text Notes 4125 5025 2    60   ~ 12
 SWD pins
 Text GLabel 4750 2400 0    60   BiDi ~ 0
@@
 	1    0    0    -1
 $EndComp
-$Comp
-L CONN_01X08 P4
-U 1 1 5757D546
-P 5775 4275
-F 0 "P4" H 5775 4725 50  0000 C CNN
-F 1 "CONN_01X08" V 5875 4275 50  0000 C CNN
-F 2 "" H 5775 4275 50  0001 C CNN
-F 3 "" H 5775 4275 50  0000 C CNN
-	1    5775 4275
-	-1   0    0    1
-$EndComp
-$Comp
-L CONN_01X08 P1
-U 1 1 5757D54C
-P 5225 4275
-F 0 "P1" H 5225 3825 50  0000 C CNN
-F 1 "CONN_01X08" V 5325 4275 50  0000 C CNN
-F 2 "" H 5225 4275 50  0001 C CNN
-F 3 "" H 5225 4275 50  0000 C CNN
-	1    5225 4275
-	1    0    0    -1
-$EndComp
-Text Notes 4650 4350 2    60   ~ 0
+Text Notes 4700 5450 2    60   ~ 0
 SWD_DIO(PTA3)
-Text GLabel 5025 3925 0    60   Input ~ 0
+Text GLabel 5025 4125 0    60   Input ~ 0
 VBUS
-$Comp
-L +3V3 #PWR04
-U 1 1 5757ECBC
-P 4750 4125
-F 0 "#PWR04" H 4750 3975 50  0001 C CNN
-F 1 "+3V3" H 4750 4265 50  0000 C CNN
-F 2 "" H 4750 4125 50  0000 C CNN
-F 3 "" H 4750 4125 50  0000 C CNN
-	1    4750 4125
-	0    -1   -1   0
-$EndComp
-Text GLabel 5975 4025 2    60   BiDi ~ 0
+Text GLabel 5025 4525 0    60   BiDi ~ 0
 PTD7
-Text GLabel 5975 4125 2    60   BiDi ~ 0
+Text GLabel 5025 4425 0    60   BiDi ~ 0
 PTD6
+Text GLabel 5975 4225 2    60   BiDi ~ 0
+PTD4
 Text GLabel 5975 4325 2    60   BiDi ~ 0
-PTD4
+PTC7
 Text GLabel 5975 4425 2    60   BiDi ~ 0
-PTC7
+PTC6
 Text GLabel 5975 4525 2    60   BiDi ~ 0
-PTC6
+PTC5
 Text GLabel 5975 4625 2    60   BiDi ~ 0
-PTC5
-Text GLabel 5975 4925 2    60   BiDi ~ 0
 PTC4
 Text GLabel 5975 5025 2    60   BiDi ~ 0
@@
 Text GLabel 5025 5625 0    60   BiDi ~ 0
 PTA18
-Text Notes 4650 4450 2    60   ~ 0
+Text Notes 7100 5575 2    60   ~ 0
 RESET_b(PTA20)
 Text GLabel 5025 5025 0    60   BiDi ~ 0
@@
 Text GLabel 5025 5525 0    60   BiDi ~ 0
 PTA4
-Text GLabel 5025 4025 0    60   Input ~ 0
+Text GLabel 5025 4225 0    60   Input ~ 0
 VREGIN
-Text GLabel 5975 3925 2    60   BiDi ~ 0
+Text GLabel 5025 4625 0    60   BiDi ~ 0
 PTE0
 $Comp
@@
 PTA20
 $Comp
-L GND #PWR05
+L GND #PWR04
 U 1 1 57581A09
 P 2350 5375
-F 0 "#PWR05" H 2350 5125 50  0001 C CNN
+F 0 "#PWR04" H 2350 5125 50  0001 C CNN
 F 1 "GND" H 2350 5225 50  0000 C CNN
 F 2 "" H 2350 5375 50  0000 C CNN
@@
 Text GLabel 1750 5225 0    60   BiDi ~ 0
 PTA4
-Text Notes 4650 4250 2    60   ~ 0
+Text Notes 4700 5175 2    60   ~ 0
 SWD_CLK(PTA0)
 Text Notes 4700 5575 2    60   ~ 0
 NMI_b(PTA4)
 $Comp
-L +3V3 #PWR08
+L +3V3 #PWR05
 U 1 1 57583F2E
 P 4750 4925
-F 0 "#PWR08" H 4750 4775 50  0001 C CNN
+F 0 "#PWR05" H 4750 4775 50  0001 C CNN
 F 1 "+3V3" H 4750 5065 50  0000 C CNN
 F 2 "" H 4750 4925 50  0000 C CNN
@@
 $EndComp
 $Comp
-L PWR_FLAG #FLG09
+L PWR_FLAG #FLG06
 U 1 1 57584EEC
 P 2950 2100
-F 0 "#FLG09" H 2950 2195 50  0001 C CNN
+F 0 "#FLG06" H 2950 2195 50  0001 C CNN
 F 1 "PWR_FLAG" H 2950 2280 50  0000 C CNN
 F 2 "" H 2950 2100 50  0000 C CNN
@@
 	2350 4925 2350 5375
 Connection ~ 2350 5225
-Wire Wire Line
-	5025 4525 4725 4525
-Text GLabel 5975 4225 2    60   BiDi ~ 0
+Text GLabel 5025 4325 0    60   BiDi ~ 0
 PTD5
-Wire Wire Line
-	5025 4125 4750 4125
-$Comp
-L GND #PWR06
+$Comp
+L GND #PWR07
 U 1 1 57582552
-P 4725 4525
-F 0 "#PWR06" H 4725 4275 50  0001 C CNN
-F 1 "GND" H 4725 4375 50  0000 C CNN
-F 2 "" H 4725 4525 50  0000 C CNN
-F 3 "" H 4725 4525 50  0000 C CNN
-	1    4725 4525
-	0    1    1    0
+P 6275 4925
+F 0 "#PWR07" H 6275 4675 50  0001 C CNN
+F 1 "GND" H 6275 4775 50  0000 C CNN
+F 2 "" H 6275 4925 50  0000 C CNN
+F 3 "" H 6275 4925 50  0000 C CNN
+	1    6275 4925
+	0    -1   -1   0
 $EndComp
 Wire Wire Line
 	5025 4925 4750 4925
-Text GLabel 5025 4425 0    60   BiDi ~ 0
-PTA20
-Text GLabel 5025 4325 0    60   BiDi ~ 0
-PTA3
-Text GLabel 5025 4225 0    60   BiDi ~ 0
-PTA0
+Wire Wire Line
+	5975 4925 6275 4925
+$Comp
+L GND #PWR08
+U 1 1 57811479
+P 6275 4125
+F 0 "#PWR08" H 6275 3875 50  0001 C CNN
+F 1 "GND" H 6275 3975 50  0000 C CNN
+F 2 "" H 6275 4125 50  0000 C CNN
+F 3 "" H 6275 4125 50  0000 C CNN
+	1    6275 4125
+	0    -1   -1   0
+$EndComp
+Wire Wire Line
+	5975 4125 6275 4125
+$Comp
+L CONN_01X06 P4
+U 1 1 578115F5
+P 5775 4375
+F 0 "P4" H 5775 4725 50  0000 C CNN
+F 1 "CONN_01X06" V 5875 4375 50  0000 C CNN
+F 2 "" H 5775 4375 50  0000 C CNN
+F 3 "" H 5775 4375 50  0000 C CNN
+	1    5775 4375
+	-1   0    0    1
+$EndComp
+$Comp
+L CONN_01X06 P1
+U 1 1 578116BA
+P 5225 4375
+F 0 "P1" H 5225 4725 50  0000 C CNN
+F 1 "CONN_01X06" V 5325 4375 50  0000 C CNN
+F 2 "" H 5225 4375 50  0000 C CNN
+F 3 "" H 5225 4375 50  0000 C CNN
+	1    5225 4375
+	1    0    0    -1
+$EndComp
 $EndSCHEMATC
