File: KL27Z_breakout.sch (KiCad schematic (older format))
At the start: 15 parts, among them J1 USB_mini_micro_B, P1 CONN_01X06, P2 CONN_01X08, P3 CONN_01X08, P4 CONN_01X06, SW1 SW_PUSH, SW2 SW_PUSH, U1 MKL27Z256VFM4

Commit message: Save 300mil work
Parts:
- C1, C2, C3, C4: footprint (none) -> keyboard_parts:C_1608
- J1: footprint (none) -> keyboard_parts:USB_miniB
- P1, P4: footprint (none) -> Pin_Headers:Pin_Header_Straight_1x06
- P2, P3: footprint (none) -> Pin_Headers:Pin_Header_Straight_1x08
- R1, R2: footprint (none) -> keyboard_parts:R_1608
- SJ1: footprint (none) -> keyboard_parts:SOLDER_JUMPER_2_WIRED
- SW1, SW2: footprint (none) -> keyboard_parts:SW_ALPS_SKRP
- U1: footprint (none) -> Housings_DFN_QFN:QFN-32-1EP_5x5mm_Pitch0.5mm
Changed lines of the file:
@@
 F 0 "U1" H 5400 3250 60  0000 C CNN
 F 1 "MKL27Z256VFM4" H 5400 1450 60  0000 C CNN
-F 2 "" H 5400 1350 60  0001 C CNN
+F 2 "Housings_DFN_QFN:QFN-32-1EP_5x5mm_Pitch0.5mm" H 5400 1350 60  0001 C CNN
 F 3 "" H 5400 1350 60  0000 C CNN
 	1    5400 2350
@@
 F 0 "J1" H 1300 1800 60  0000 C CNN
 F 1 "USB_mini_micro_B" H 1550 2100 60  0001 C CNN
-F 2 "" H 1650 1850 60  0001 C CNN
+F 2 "keyboard_parts:USB_miniB" H 1650 1850 60  0001 C CNN
 F 3 "" H 1650 1850 60  0000 C CNN
 	1    1700 1850
@@
 F 0 "R1" V 3275 1800 50  0000 C CNN
 F 1 "33" V 3350 1800 50  0000 C CNN
-F 2 "" V 3280 1800 50  0001 C CNN
+F 2 "keyboard_parts:R_1608" V 3280 1800 50  0001 C CNN
 F 3 "" H 3350 1800 50  0000 C CNN
 	1    3350 1800
@@
 F 0 "R2" V 3430 1900 50  0000 C CNN
 F 1 "33" V 3350 1900 50  0000 C CNN
-F 2 "" V 3280 1900 50  0001 C CNN
+F 2 "keyboard_parts:R_1608" V 3280 1900 50  0001 C CNN
 F 3 "" H 3350 1900 50  0000 C CNN
 	1    3350 1900
@@
 F 0 "C2" H 3325 3250 50  0000 L CNN
 F 1 "2.2u" H 3325 3050 50  0000 L CNN
-F 2 "" H 3338 3000 50  0001 C CNN
+F 2 "keyboard_parts:C_1608" H 3338 3000 50  0001 C CNN
 F 3 "" H 3300 3150 50  0000 C CNN
 	1    3300 3150
@@
 F 0 "C1" H 2975 3250 50  0000 L CNN
 F 1 "4.7u" H 2975 3050 50  0000 L CNN
-F 2 "" H 2988 3000 50  0001 C CNN
+F 2 "keyboard_parts:C_1608" H 2988 3000 50  0001 C CNN
 F 3 "" H 2950 3150 50  0000 C CNN
 	1    2950 3150
@@
 F 0 "C4" H 4025 3250 50  0000 L CNN
 F 1 "0.1u" H 4025 3050 50  0000 L CNN
-F 2 "" H 4038 3000 50  0001 C CNN
+F 2 "keyboard_parts:C_1608" H 4038 3000 50  0001 C CNN
 F 3 "" H 4000 3150 50  0000 C CNN
 	1    4000 3150
@@
 F 0 "C3" H 3675 3250 50  0000 L CNN
 F 1 "0.1u" H 3675 3050 50  0000 L CNN
-F 2 "" H 3688 3000 50  0001 C CNN
+F 2 "keyboard_parts:C_1608" H 3688 3000 50  0001 C CNN
 F 3 "" H 3650 3150 50  0000 C CNN
 	1    3650 3150
@@
 F 0 "SJ1" H 1825 3875 60  0000 C CNN
 F 1 "SOLDER_JUMPER" H 1875 4075 60  0001 C CNN
-F 2 "" H 1875 3925 60  0001 C CNN
+F 2 "keyboard_parts:SOLDER_JUMPER_2_WIRED" H 1875 3925 60  0001 C CNN
 F 3 "" H 1875 3925 60  0000 C CNN
 	1    1825 3925
@@
 F 0 "P3" H 5775 5725 50  0000 C CNN
 F 1 "CONN_01X08" V 5875 5275 50  0000 C CNN
-F 2 "" H 5775 5275 50  0001 C CNN
+F 2 "Pin_Headers:Pin_Header_Straight_1x08" H 5775 5275 50  0001 C CNN
 F 3 "" H 5775 5275 50  0000 C CNN
 	1    5775 5275
@@
 F 0 "P2" H 5225 4800 50  0000 C CNN
 F 1 "CONN_01X08" V 5325 5275 50  0000 C CNN
-F 2 "" H 5225 5275 50  0001 C CNN
+F 2 "Pin_Headers:Pin_Header_Straight_1x08" H 5225 5275 50  0001 C CNN
 F 3 "" H 5225 5275 50  0000 C CNN
 	1    5225 5275
@@
 F 0 "SW1" H 2200 5035 50  0000 C CNN
 F 1 "SW_PUSH" H 2050 4845 50  0000 C CNN
-F 2 "" H 2050 4925 50  0001 C CNN
+F 2 "keyboard_parts:SW_ALPS_SKRP" H 2050 4925 50  0001 C CNN
 F 3 "" H 2050 4925 50  0000 C CNN
 	1    2050 4925
@@
 F 0 "SW2" H 2200 5335 50  0000 C CNN
 F 1 "SW_PUSH" H 2050 5145 50  0000 C CNN
-F 2 "" H 2050 5225 50  0001 C CNN
+F 2 "keyboard_parts:SW_ALPS_SKRP" H 2050 5225 50  0001 C CNN
 F 3 "" H 2050 5225 50  0000 C CNN
 	1    2050 5225
@@
 F 0 "P4" H 5775 4725 50  0000 C CNN
 F 1 "CONN_01X06" V 5875 4375 50  0000 C CNN
-F 2 "" H 5775 4375 50  0000 C CNN
+F 2 "Pin_Headers:Pin_Header_Straight_1x06" H 5775 4375 50  0001 C CNN
 F 3 "" H 5775 4375 50  0000 C CNN
 	1    5775 4375
@@
 F 0 "P1" H 5225 4725 50  0000 C CNN
 F 1 "CONN_01X06" V 5325 4375 50  0000 C CNN
-F 2 "" H 5225 4375 50  0000 C CNN
+F 2 "Pin_Headers:Pin_Header_Straight_1x06" H 5225 4375 50  0001 C CNN
 F 3 "" H 5225 4375 50  0000 C CNN
 	1    5225 4375
