File: KL27Z_breakout.sch (KiCad schematic (older format))
At the start: 15 parts, among them J1 USB_mini_micro_B, P1 CONN_01X06, P2 CONN_01X08, P3 CONN_01X08, P4 CONN_01X06, SW1 SW_PUSH, SW2 SW_PUSH, U1 MKL27Z256VFM4

Commit message: Add silk screen fill under thermal pad
Parts:
- removed P1, P4: CONN_01X06, Pin_Headers:Pin_Header_Straight_1x06, symbol CONN_01X06
- added P1, P4: CONN_01X08, symbol CONN_01X08
- C1, C2, C3, C4: footprint keyboard_parts:C_1608 -> (none)
- J1: footprint keyboard_parts:USB_miniB -> (none)
- P2, P3: footprint Pin_Headers:Pin_Header_Straight_1x08 -> (none)
- R1, R2: footprint keyboard_parts:R_1608 -> (none)
- SJ1: footprint keyboard_parts:SOLDER_JUMPER_2_WIRED -> (none)
- SW1, SW2: footprint keyboard_parts:SW_ALPS_SKRP -> (none)
- U1: footprint Housings_DFN_QFN:QFN-32-1EP_5x5mm_Pitch0.5mm -> (none); symbol MKL27Z256VFM4-RESCUE-KL27Z_breakout -> MKL27Z256VFM4
Connections:
- net +3V3: now also P1.3 (P3)
- net GND: now also P2.8 (P8), P1.7 (P7); no longer P3.8 (P8)
- net PTA0: now also P1.4 (P4)
- net PTA18: now also P3.1 (P1); no longer P2.8 (P8)
- net PTA19: now also P3.2 (P2); no longer P3.1 (P1)
- net PTA20: now also P3.3 (P3), P1.6 (P6); no longer P3.2 (P2)
- net PTA3: now also P1.5 (P5)
- net PTB0: now also P3.4 (P4); no longer P3.3 (P3)
- net PTB1: now also P3.5 (P5); no longer P3.4 (P4)
- net PTC1: now also P3.6 (P6); no longer P3.5 (P5)
- net PTC2: now also P3.7 (P7); no longer P3.6 (P6)
- net PTC3: now also P3.8 (P8); no longer P3.7 (P7)
- net PTC4: now also P4.1 (P1)
- net PTC5: now also P4.2 (P2)
- net PTC6: now also P4.3 (P3)
- net PTC7: now also P4.4 (P4)
- net PTD4: now also P4.5 (P5)
- net PTD5: now also P4.6 (P6)
- net PTD6: now also P4.7 (P7)
- net PTD7: now also P4.8 (P8)
- net PTE0: now also P1.8 (P8)
- net VBUS: now also P1.1 (P1)
- net VREGIN: now also P1.2 (P2)
Changed lines of the file:
@@
 EESchema Schematic File Version 2
-LIBS:KL27Z_breakout-rescue
 LIBS:power
 LIBS:device
@@
 LIBS:mkl27z256vfm4
 LIBS:keyboard_parts
-LIBS:KL27Z_breakout-cache
 EELAYER 25 0
 EELAYER END
@@
 $EndDescr
 $Comp
-L MKL27Z256VFM4-RESCUE-KL27Z_breakout U1
+L MKL27Z256VFM4 U1
 U 1 1 57578DE2
 P 5400 2350
 F 0 "U1" H 5400 3250 60  0000 C CNN
 F 1 "MKL27Z256VFM4" H 5400 1450 60  0000 C CNN
-F 2 "Housings_DFN_QFN:QFN-32-1EP_5x5mm_Pitch0.5mm" H 5400 1350 60  0001 C CNN
+F 2 "" H 5400 1350 60  0001 C CNN
 F 3 "" H 5400 1350 60  0000 C CNN
 	1    5400 2350
@@
 F 0 "J1" H 1300 1800 60  0000 C CNN
 F 1 "USB_mini_micro_B" H 1550 2100 60  0001 C CNN
-F 2 "keyboard_parts:USB_miniB" H 1650 1850 60  0001 C CNN
+F 2 "" H 1650 1850 60  0001 C CNN
 F 3 "" H 1650 1850 60  0000 C CNN
 	1    1700 1850
@@
 F 0 "R1" V 3275 1800 50  0000 C CNN
 F 1 "33" V 3350 1800 50  0000 C CNN
-F 2 "keyboard_parts:R_1608" V 3280 1800 50  0001 C CNN
+F 2 "" V 3280 1800 50  0001 C CNN
 F 3 "" H 3350 1800 50  0000 C CNN
 	1    3350 1800
@@
 F 0 "R2" V 3430 1900 50  0000 C CNN
 F 1 "33" V 3350 1900 50  0000 C CNN
-F 2 "keyboard_parts:R_1608" V 3280 1900 50  0001 C CNN
+F 2 "" V 3280 1900 50  0001 C CNN
 F 3 "" H 3350 1900 50  0000 C CNN
 	1    3350 1900
@@
 F 0 "C2" H 3325 3250 50  0000 L CNN
 F 1 "2.2u" H 3325 3050 50  0000 L CNN
-F 2 "keyboard_parts:C_1608" H 3338 3000 50  0001 C CNN
+F 2 "" H 3338 3000 50  0001 C CNN
 F 3 "" H 3300 3150 50  0000 C CNN
 	1    3300 3150
@@
 F 0 "C1" H 2975 3250 50  0000 L CNN
 F 1 "4.7u" H 2975 3050 50  0000 L CNN
-F 2 "keyboard_parts:C_1608" H 2988 3000 50  0001 C CNN
+F 2 "" H 2988 3000 50  0001 C CNN
 F 3 "" H 2950 3150 50  0000 C CNN
 	1    2950 3150
@@
 F 0 "C4" H 4025 3250 50  0000 L CNN
 F 1 "0.1u" H 4025 3050 50  0000 L CNN
-F 2 "keyboard_parts:C_1608" H 4038 3000 50  0001 C CNN
+F 2 "" H 4038 3000 50  0001 C CNN
 F 3 "" H 4000 3150 50  0000 C CNN
 	1    4000 3150
@@
 F 0 "C3" H 3675 3250 50  0000 L CNN
 F 1 "0.1u" H 3675 3050 50  0000 L CNN
-F 2 "keyboard_parts:C_1608" H 3688 3000 50  0001 C CNN
+F 2 "" H 3688 3000 50  0001 C CNN
 F 3 "" H 3650 3150 50  0000 C CNN
 	1    3650 3150
@@
 F 0 "SJ1" H 1825 3875 60  0000 C CNN
 F 1 "SOLDER_JUMPER" H 1875 4075 60  0001 C CNN
-F 2 "keyboard_parts:SOLDER_JUMPER_2_WIRED" H 1875 3925 60  0001 C CNN
+F 2 "" H 1875 3925 60  0001 C CNN
 F 3 "" H 1875 3925 60  0000 C CNN
 	1    1825 3925
@@
 Text Notes 1400 4175 0    60   ~ 0
 External power option
-Text Notes 4125 5025 2    60   ~ 12
+Text Notes 4050 4100 2    60   ~ 12
 SWD pins
 Text GLabel 4750 2400 0    60   BiDi ~ 0
@@
 F 0 "P3" H 5775 5725 50  0000 C CNN
 F 1 "CONN_01X08" V 5875 5275 50  0000 C CNN
-F 2 "Pin_Headers:Pin_Header_Straight_1x08" H 5775 5275 50  0001 C CNN
+F 2 "" H 5775 5275 50  0001 C CNN
 F 3 "" H 5775 5275 50  0000 C CNN
 	1    5775 5275
@@
 F 0 "P2" H 5225 4800 50  0000 C CNN
 F 1 "CONN_01X08" V 5325 5275 50  0000 C CNN
-F 2 "Pin_Headers:Pin_Header_Straight_1x08" H 5225 5275 50  0001 C CNN
+F 2 "" H 5225 5275 50  0001 C CNN
 F 3 "" H 5225 5275 50  0000 C CNN
 	1    5225 5275
 	1    0    0    -1
 $EndComp
-Text Notes 4700 5450 2    60   ~ 0
+$Comp
+L CONN_01X08 P4
+U 1 1 5757D546
+P 5775 4275
+F 0 "P4" H 5775 4725 50  0000 C CNN
+F 1 "CONN_01X08" V 5875 4275 50  0000 C CNN
+F 2 "" H 5775 4275 50  0001 C CNN
+F 3 "" H 5775 4275 50  0000 C CNN
+	1    5775 4275
+	-1   0    0    1
+$EndComp
+$Comp
+L CONN_01X08 P1
+U 1 1 5757D54C
+P 5225 4275
+F 0 "P1" H 5225 3825 50  0000 C CNN
+F 1 "CONN_01X08" V 5325 4275 50  0000 C CNN
+F 2 "" H 5225 4275 50  0001 C CNN
+F 3 "" H 5225 4275 50  0000 C CNN
+	1    5225 4275
+	1    0    0    -1
+$EndComp
+Text Notes 4650 4350 2    60   ~ 0
 SWD_DIO(PTA3)
-Text GLabel 5025 4125 0    60   Input ~ 0
+Text GLabel 5025 3925 0    60   Input ~ 0
 VBUS
-Text GLabel 5025 4525 0    60   BiDi ~ 0
+$Comp
+L +3V3 #PWR04
+U 1 1 5757ECBC
+P 4750 4125
+F 0 "#PWR04" H 4750 3975 50  0001 C CNN
+F 1 "+3V3" H 4750 4265 50  0000 C CNN
+F 2 "" H 4750 4125 50  0000 C CNN
+F 3 "" H 4750 4125 50  0000 C CNN
+	1    4750 4125
+	0    -1   -1   0
+$EndComp
+Text GLabel 5975 3925 2    60   BiDi ~ 0
 PTD7
-Text GLabel 5025 4425 0    60   BiDi ~ 0
+Text GLabel 5975 4025 2    60   BiDi ~ 0
 PTD6
 Text GLabel 5975 4225 2    60   BiDi ~ 0
@@
 Text GLabel 5975 4625 2    60   BiDi ~ 0
 PTC4
+Text GLabel 5975 4925 2    60   BiDi ~ 0
+PTC3
 Text GLabel 5975 5025 2    60   BiDi ~ 0
-PTC3
+PTC2
 Text GLabel 5975 5125 2    60   BiDi ~ 0
-PTC2
+PTC1
 Text GLabel 5975 5225 2    60   BiDi ~ 0
-PTC1
+PTB1
 Text GLabel 5975 5325 2    60   BiDi ~ 0
-PTB1
+PTB0
 Text GLabel 5975 5425 2    60   BiDi ~ 0
-PTB0
+PTA20
 Text GLabel 5975 5525 2    60   BiDi ~ 0
-PTA20
+PTA19
 Text GLabel 5975 5625 2    60   BiDi ~ 0
-PTA19
-Text GLabel 5025 5625 0    60   BiDi ~ 0
 PTA18
-Text Notes 7100 5575 2    60   ~ 0
+Text Notes 4650 4450 2    60   ~ 0
 RESET_b(PTA20)
 Text GLabel 5025 5025 0    60   BiDi ~ 0
@@
 Text GLabel 5025 5525 0    60   BiDi ~ 0
 PTA4
-Text GLabel 5025 4225 0    60   Input ~ 0
+Text GLabel 5025 4025 0    60   Input ~ 0
 VREGIN
 Text GLabel 5025 4625 0    60   BiDi ~ 0
@@
 F 0 "SW1" H 2200 5035 50  0000 C CNN
 F 1 "SW_PUSH" H 2050 4845 50  0000 C CNN
-F 2 "keyboard_parts:SW_ALPS_SKRP" H 2050 4925 50  0001 C CNN
+F 2 "" H 2050 4925 50  0001 C CNN
 F 3 "" H 2050 4925 50  0000 C CNN
 	1    2050 4925
@@
 PTA20
 $Comp
-L GND #PWR04
+L GND #PWR05
 U 1 1 57581A09
 P 2350 5375
-F 0 "#PWR04" H 2350 5125 50  0001 C CNN
+F 0 "#PWR05" H 2350 5125 50  0001 C CNN
 F 1 "GND" H 2350 5225 50  0000 C CNN
 F 2 "" H 2350 5375 50  0000 C CNN
@@
 F 0 "SW2" H 2200 5335 50  0000 C CNN
 F 1 "SW_PUSH" H 2050 5145 50  0000 C CNN
-F 2 "keyboard_parts:SW_ALPS_SKRP" H 2050 5225 50  0001 C CNN
+F 2 "" H 2050 5225 50  0001 C CNN
 F 3 "" H 2050 5225 50  0000 C CNN
 	1    2050 5225
@@
 Text GLabel 1750 5225 0    60   BiDi ~ 0
 PTA4
-Text Notes 4700 5175 2    60   ~ 0
+Text GLabel 5025 4225 0    60   BiDi ~ 0
+PTA0
+Text GLabel 5025 4325 0    60   BiDi ~ 0
+PTA3
+Text GLabel 5025 4425 0    60   BiDi ~ 0
+PTA20
+$Comp
+L GND #PWR06
+U 1 1 57582552
+P 4725 4525
+F 0 "#PWR06" H 4725 4275 50  0001 C CNN
+F 1 "GND" H 4725 4375 50  0000 C CNN
+F 2 "" H 4725 4525 50  0000 C CNN
+F 3 "" H 4725 4525 50  0000 C CNN
+	1    4725 4525
+	0    1    1    0
+$EndComp
+Text Notes 4650 4250 2    60   ~ 0
 SWD_CLK(PTA0)
+$Comp
+L GND #PWR07
+U 1 1 5758372E
+P 4750 5625
+F 0 "#PWR07" H 4750 5375 50  0001 C CNN
+F 1 "GND" H 4750 5475 50  0000 C CNN
+F 2 "" H 4750 5625 50  0000 C CNN
+F 3 "" H 4750 5625 50  0000 C CNN
+	1    4750 5625
+	0    1    1    0
+$EndComp
 Text Notes 4700 5575 2    60   ~ 0
 NMI_b(PTA4)
 $Comp
-L +3V3 #PWR05
+L +3V3 #PWR08
 U 1 1 57583F2E
 P 4750 4925
-F 0 "#PWR05" H 4750 4775 50  0001 C CNN
+F 0 "#PWR08" H 4750 4775 50  0001 C CNN
 F 1 "+3V3" H 4750 5065 50  0000 C CNN
 F 2 "" H 4750 4925 50  0000 C CNN
@@
 $EndComp
 $Comp
-L PWR_FLAG #FLG06
+L PWR_FLAG #FLG09
 U 1 1 57584EEC
 P 2950 2100
-F 0 "#FLG06" H 2950 2195 50  0001 C CNN
+F 0 "#FLG09" H 2950 2195 50  0001 C CNN
 F 1 "PWR_FLAG" H 2950 2280 50  0000 C CNN
 F 2 "" H 2950 2100 50  0000 C CNN
@@
 Connection ~ 3300 3350
 Wire Wire Line
+	5025 4125 4750 4125
+Wire Wire Line
 	3300 2000 3300 3000
 Wire Wire Line
 	2350 4925 2350 5375
 Connection ~ 2350 5225
-Text GLabel 5025 4325 0    60   BiDi ~ 0
+Wire Wire Line
+	5025 4525 4725 4525
+Wire Wire Line
+	5025 5625 4750 5625
+Wire Wire Line
+	5025 4925 4750 4925
+Text GLabel 5975 4125 2    60   BiDi ~ 0
 PTD5
-$Comp
-L GND #PWR07
-U 1 1 57582552
-P 6275 4925
-F 0 "#PWR07" H 6275 4675 50  0001 C CNN
-F 1 "GND" H 6275 4775 50  0000 C CNN
-F 2 "" H 6275 4925 50  0000 C CNN
-F 3 "" H 6275 4925 50  0000 C CNN
-	1    6275 4925
-	0    -1   -1   0
-$EndComp
-Wire Wire Line
-	5025 4925 4750 4925
-Wire Wire Line
-	5975 4925 6275 4925
-$Comp
-L GND #PWR08
-U 1 1 57811479
-P 6275 4125
-F 0 "#PWR08" H 6275 3875 50  0001 C CNN
-F 1 "GND" H 6275 3975 50  0000 C CNN
-F 2 "" H 6275 4125 50  0000 C CNN
-F 3 "" H 6275 4125 50  0000 C CNN
-	1    6275 4125
-	0    -1   -1   0
-$EndComp
-Wire Wire Line
-	5975 4125 6275 4125
-$Comp
-L CONN_01X06 P4
-U 1 1 578115F5
-P 5775 4375
-F 0 "P4" H 5775 4725 50  0000 C CNN
-F 1 "CONN_01X06" V 5875 4375 50  0000 C CNN
-F 2 "Pin_Headers:Pin_Header_Straight_1x06" H 5775 4375 50  0001 C CNN
-F 3 "" H 5775 4375 50  0000 C CNN
-	1    5775 4375
-	-1   0    0    1
-$EndComp
-$Comp
-L CONN_01X06 P1
-U 1 1 578116BA
-P 5225 4375
-F 0 "P1" H 5225 4725 50  0000 C CNN
-F 1 "CONN_01X06" V 5325 4375 50  0000 C CNN
-F 2 "Pin_Headers:Pin_Header_Straight_1x06" H 5225 4375 50  0001 C CNN
-F 3 "" H 5225 4375 50  0000 C CNN
-	1    5225 4375
-	1    0    0    -1
-$EndComp
 $EndSCHEMATC
